File: circuit/remote_controller/remote_controller.kicad_sch (KiCad schematic)
At the start: 68 parts, among them J1 Conn_01x02_Male, J2 USB_C_Receptacle_USB2.0, Q1 SS8050-G, Q2 SS8050-G, SW1 SW_Push, SW10 SW_Push, SW2 SW_Push, SW3 SW_Push, SW4 SW_Push, SW5 SW_Push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

Commit message: Added csv file.
Parts:
- SW1, SW2: Vendor (none) -> https://www.mouser.jp/ProductDetail/CK/KMR231NGLFS?qs=sb%25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
- SW10, SW3, SW4, SW5, SW6, SW7, SW8, SW9: Vendor (none) -> https://www.mouser.jp/ProductDetail/Diptronics/DTSM-65N-V-B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
Changed lines of the file:
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@@
+      (effects (font (size 1.27 1.27)) hide)
+    )
+    (property "Vendor" "https://www.mouser.jp/ProductDetail/Diptronics/DTSM-65N-V-B?qs=gTYE2QTfZfSXwXAGPNekUg%3D%3D" (id 4) (at 262.89 41.91 0)
       (effects (font (size 1.27 1.27)) hide)
     )
@@
       (effects (font (size 1.27 1.27)) hide)
     )
+    (property "Vendor" "https://www.mouser.jp/ProductDetail/Diptronics/DTSM-65N-V-B?qs=gTYE2QTfZfSXwXAGPNekUg%3D%3D" (id 4) (at 262.89 105.41 0)
+      (effects (font (size 1.27 1.27)) hide)
+    )
     (pin "1")
     (pin "2")
@@
       (effects (font (size 1.27 1.27)) hide)
     )
+    (property "Vendor" "https://www.mouser.jp/ProductDetail/Diptronics/DTSM-65N-V-B?qs=gTYE2QTfZfSXwXAGPNekUg%3D%3D" (id 4) (at 222.25 105.41 0)
+      (effects (font (size 1.27 1.27)) hide)
+    )
     (pin "1")
     (pin "2")
@@
       (effects (font (size 1.27 1.27)) hide)
     )
+    (property "Vendor" "https://www.mouser.jp/ProductDetail/Diptronics/DTSM-65N-V-B?qs=gTYE2QTfZfSXwXAGPNekUg%3D%3D" (id 4) (at 222.25 137.16 0)
+      (effects (font (size 1.27 1.27)) hide)
+    )
     (pin "1")
     (pin "2")
@@
       (effects (font (size 1.27 1.27)) hide)
     )
+    (property "Vendor" "https://www.mouser.jp/ProductDetail/Diptronics/DTSM-65N-V-B?qs=gTYE2QTfZfSXwXAGPNekUg%3D%3D" (id 4) (at 222.25 41.91 0)
+      (effects (font (size 1.27 1.27)) hide)
+    )
     (pin "1")
     (pin "2")
@@
       (effects (font (size 1.27 1.27)) hide)
     )
+    (property "Vendor" "https://www.mouser.jp/ProductDetail/Diptronics/DTSM-65N-V-B?qs=gTYE2QTfZfSXwXAGPNekUg%3D%3D" (id 4) (at 262.89 137.16 0)
+      (effects (font (size 1.27 1.27)) hide)
+    )
     (pin "1")
     (pin "2")
@@
       (effects (font (size 1.27 1.27)) hide)
     )
+    (property "Vendor" "https://www.mouser.jp/ProductDetail/CK/KMR231NGLFS?qs=sb%252But3Lm4x1Y5NsXXdZx2g%3D%3D" (id 4) (at 76.2 144.78 0)
+      (effects (font (size 1.27 1.27)) hide)
+    )
     (pin "1")
     (pin "2")
@@
     )
     (property "Datasheet" "~" (id 3) (at 267.97 73.66 0)
+      (effects (font (size 1.27 1.27)) hide)
+    )
+    (property "Vendor" "https://www.mouser.jp/ProductDetail/Diptronics/DTSM-65N-V-B?qs=gTYE2QTfZfSXwXAGPNekUg%3D%3D" (id 4) (at 262.89 73.66 0)
       (effects (font (size 1.27 1.27)) hide)
     )
@@
       (effects (font (size 1.27 1.27)) hide)
     )
+    (property "Vendor" "https://www.mouser.jp/ProductDetail/CK/KMR231NGLFS?qs=sb%252But3Lm4x1Y5NsXXdZx2g%3D%3D" (id 4) (at 77.47 173.99 0)
+      (effects (font (size 1.27 1.27)) hide)
+    )
     (pin "1")
     (pin "2")
@@
       (effects (font (size 1.27 1.27)) hide)
     )
+    (property "Vendor" "https://www.mouser.jp/ProductDetail/Diptronics/DTSM-65N-V-B?qs=gTYE2QTfZfSXwXAGPNekUg%3D%3D" (id 4) (at 222.25 73.66 0)
+      (effects (font (size 1.27 1.27)) hide)
+    )
