File: circuit/omni_wheel/omni_wheel.kicad_sch (KiCad schematic)
At the start: 48 parts, among them J1 Conn_01x02_Male, J2 USB_C_Receptacle_USB2.0, Q1 SS8050-G, Q2 SS8050-G, SW1 SW_Push, SW2 SW_Push, SW3 SW_Push, SW4 SW_SPDT, U1 LT1963AxST-3.3, U2 ESP32-WROVER-B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

Commit message: connect nsleep to high and remove unnecessary switch (2/2).
Parts:
- removed D5: 1N4148W, Diode_SMD:D_SOD-123, symbol Diode:1N4148W
- removed SW4: SW_SPDT, Button_Switch_THT:SW_Slide_1P2T_CK_OS102011MS2Q, symbol Switch:SW_SPDT
- J1: Vendor (none) -> https://www.digikey.jp/ja/products/detail/adam-tech/PH1RB-0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
Connections:
- no-connect marks 32 -> 31
Other:
- moved on the sheet: C1, C6, D1, R3, U1
